File: hardware/kicad/module-I2C-buzzer.kicad_sch (KiCad schematic)
At the start: 15 parts, among them J1 JST 4 Pin Qwiic I2C Connector, J2 JST 4 Pin Qwiic I2C Connector, J3 noknok_FlashPads_I2C-module, Q1 MMBT3904, U1 CH32V003J4M6

Commit message: hardware: update schematic, rename BOM file, refresh schematic PDF and fix readme links
Other:
- note added: "noknok Module I2C Buzzer"
- note removed: "I2C Buzzer"
- note removed: "Specs: - I2C powered at 3.3V"
